Commit message: removing untested elements for kinetic

File: summit_xls_ur5_description/robots/summit_xls_ur5_omni.urdf.xacro (robot description, xacro)
@@ -12,21 +12,11 @@
 	<xacro:property name="hq" value="true" />
 	<!-- Import Summit XL Steel -->
-	<xacro:include filename="$(find summit_xl_description)/robots/summit_xl_hls_omni.urdf.xacro"/>
+	<xacro:include filename="$(find summit_xl_description)/robots/summit_xls_std.urdf.xacro"/>
 	<!-- Import UR5 arm -->
 	<xacro:include filename="$(find ur_description)/urdf/ur5.urdf.xacro" />
-	<!-- SENSORS -->
-    <!-- xacro:sensor_sick_s300 name="laser_front" parent="base_link">
-		<origin xyz="${front_laser_offset_x} ${front_laser_offset_y} ${front_laser_offset_z}" rpy="0 0 ${-PI/4.0}"/>
-	</xacro:sensor_sick_s300 -->
-    <!-- xacro:BB2-08S2C-38 frame="bumblebee2" name="bumblebee2" />
-		<joint name="world_camera_joint" type="fixed">
-			<origin xyz="0.325 0 0.210" rpy="0 0 0" />
-            <parent link="base_link" />
-         <child link="bumblebee2" />
-    </joint -->
 	<!-- UR5 Arm -->
-    <xacro:ur5_robot prefix="arm_" joint_limited="true">
+    <xacro:ur5_robot prefix="$(prefix)arm_" joint_limited="true">
     </xacro:ur5_robot>
-    <joint name="arm_base_joint" type="fixed">
+    <joint name="$(prefix)arm_base_joint" type="fixed">
 		<origin xyz="0.175 0 0.303" rpy="0 0 0" />
 		<parent link="base_link" />
